File: power.kicad_sch (KiCad schematic)
At the start: 0 parts

Commit message: Add LM5156 flyback controller symbol
And add it to the power sheet. This will be the controller for the 12 V
to 170 V DC-DC converter.
Parts:
- added U?: LM5156, symbol nixies:LM5156
Changed lines of the file:
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@@
 (kicad_sch (version 20211123) (generator eeschema)
   (paper "A4")
+  (symbol (lib_id "nixies:LM5156") (at 77.47 53.34 0) (unit 1)
+    (in_bom yes) (on_board yes) (fields_autoplaced)
+    (property "Reference" "U?" (id 0) (at 83.185 45.72 0))
+    (property "Value" "LM5156" (id 1) (at 83.185 48.26 0))
+    (property "Footprint" "" (id 2) (at 77.47 53.34 0)
+      (effects (font (size 1.27 1.27)) hide)
+    )
+    (property "Datasheet" "" (id 3) (at 77.47 53.34 0)
+      (effects (font (size 1.27 1.27)) hide)
+    )
+    (pin "1")
+    (pin "10")
+    (pin "11")
+    (pin "12")
+    (pin "13")
+    (pin "14")
+    (pin "2")
+    (pin "3")
+    (pin "4")
+    (pin "5")
+    (pin "6")
+    (pin "7")
+    (pin "8")
+    (pin "9")
+  )
 )
